File: pcb/keypad/keypad.kicad_pcb (KiCad board)
At the start: 2 copper layers, 22 parts, among them SW1 SW_Push, SW10 Enc1, SW11 Enc2, SW12 Reset, SW2 SW_Push, SW3 SW_Push, SW4 SW_Push, SW5 SW_Push, SW6 SW_Push, SW7 SW_Push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

Commit message: 更新 kicad
Parts:
- moved SW11 31.6 mm to (163.1, 57.5)
- moved SW10 30.4 mm to (133.5, 46.5)
- moved D8 23.2 mm to (163.0, 75.5), turned to 0 degrees
- moved D4 22.8 mm to (163.7, 94.5), turned to 0 degrees
- moved SW4 19.0 mm to (167.0, 104.0)
- moved SW8 19.0 mm to (167.0, 85.0)
- moved D3 14.3 mm to (143.0, 75.5), turned to 0 degrees
- moved D7 5.19 mm to (152.1, 94.5)
- moved D2 3.81 mm to (134.5, 75.5)
- moved SW12 2.26 mm to (124.5, 24.5)
- moved SW9 0.50 mm to (135.0, 62.5)
Routing:
- net C: track 0.00 -> 205.3 mm
- net B: track 0.00 -> 120.6 mm
- net X: track 0.00 -> 110.3 mm
- net GND: track 0.00 -> 99.6 mm
- net Y: track 0.00 -> 90.0 mm
- net Z: track 0.00 -> 73.4 mm
- net A: track 0.00 -> 71.1 mm
- net ROT2B: track 0.00 -> 57.8 mm
- net ROT2A: track 0.00 -> 51.0 mm
- net Net-(D7-Pad2): track 0.00 -> 29.9 mm
- net ROT1B: track 0.00 -> 24.2 mm
- net ROT1A: track 0.00 -> 18.2 mm
- net Net-(D9-Pad2): track 0.00 -> 12.8 mm
- net reset: track 0.00 -> 12.5 mm
- net Net-(D2-Pad2): track 0.00 -> 6.47 mm
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
Commit message: 変更 pcb
Parts:
- added REF: MountingHole_3.5mm_Pad_TopBottom, MountingHole:MountingHole_3.5mm_Pad_TopBottom, F.Cu at (197.4, 54.0)
- added REF**: MountingHole_3.5mm_Pad_TopBottom, MountingHole:MountingHole_3.5mm_Pad_TopBottom, F.Cu at (109.4, 54.0)
- added REF**: MountingHole_3.5mm_Pad_TopBottom, MountingHole:MountingHole_3.5mm_Pad_TopBottom, F.Cu at (197.4, 142.0)
- added REF**: MountingHole_3.5mm_Pad_TopBottom, MountingHole:MountingHole_3.5mm_Pad_TopBottom, F.Cu at (109.4, 142.0)
- moved D3 33.4 mm to (158.6, 105.0)
- moved D7 32.8 mm to (166.5, 124.0)
- moved D8 32.8 mm to (177.4, 105.0)
- moved D9 32.8 mm to (139.4, 93.8)
- moved SW1 32.8 mm to (124.4, 114.5)
- moved SW10 32.8 mm to (147.9, 76.0)
- moved SW11 32.8 mm to (177.5, 87.0)
- moved SW12 32.8 mm to (138.9, 54.0)
- moved SW2 32.8 mm to (143.4, 114.5)
- moved SW3 32.8 mm to (162.4, 114.5)
- moved SW4 32.8 mm to (181.4, 133.5)
- moved SW5 32.8 mm to (124.4, 133.5)
- moved SW6 32.8 mm to (143.4, 133.5)
- moved SW7 32.8 mm to (162.4, 133.5)
- moved SW8 32.8 mm to (181.4, 114.5)
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Routing:
- net Net-(D7-Pad2): track 29.9 -> 7.87 mm
- net B: track 120.6 -> 106.4 mm
- net Net-(D6-Pad2): track 4.77 -> 14.4 mm
- net reset: track 12.5 -> 19.0 mm
- net Y: track 90.0 -> 96.2 mm
- net Z: track 73.4 -> 79.3 mm
- net X: track 110.3 -> 115.7 mm
- net Net-(D1-Pad2): track 4.72 -> 8.16 mm
- net Net-(D5-Pad2): track 4.77 -> 8.18 mm
- net GND: track 99.6 -> 102.2 mm
- net C: track 205.3 -> 207.5 mm
- net A: track 71.1 -> 69.1 mm
- net Net-(D2-Pad2): track 6.47 -> 8.16 mm
- net ROT1A: track 18.2 -> 18.7 mm
- added copper zone on B.Cu, net GND
- added copper zone on F.Cu, net GND
Other:
- board outline added: 100 x 100 mm
- rule pad_to_mask_clearance: 0 -> 0.05

Commit message: 変更 pcb
Other:
- board text added: "JLCJLCJLCJLC"
- board text added: "KEYPAD-MIST"
- board text added: "R3-333"
- board text added: "VRLAB-KC"
Changed lines of the file:
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@@
   (gr_line (start 131.38 120.5) (end 131.38 121.5) (layer "F.SilkS") (width 0.15))
   (gr_line (start 131.38 107.5) (end 131.38 108.5) (layer "F.SilkS") (width 0.15))
+  (gr_circle (center 170.5 54.5) (end 171 57) (layer "F.SilkS") (width 0.15) (fill none))
   (gr_line (start 174.38 120.5) (end 174.38 121.5) (layer "F.SilkS") (width 0.15))
   (gr_line (start 117.38 139.5) (end 117.38 140.5) (layer "F.SilkS") (width 0.15))
@@
   (gr_circle (center 151.5 69) (end 162.5 69) (layer "Dwgs.User") (width 0.15) (fill none))
   (gr_rect (start 103.38 48) (end 203.38 148) (layer "Edge.Cuts") (width 0.1) (fill none))
+  (gr_text "KEYPAD-MIST" (at 154.5 54) (layer "F.SilkS")
+    (effects (font (size 2 1.8) (thickness 0.3)))
+  )
+  (gr_text "R3-333" (at 183 56.5) (layer "F.SilkS")
+    (effects (font (size 1.5 1.5) (thickness 0.3)))
+  )
+  (gr_text "JLCJLCJLCJLC" (at 183.5 144) (layer "F.SilkS")
+    (effects (font (size 1.5 1.5) (thickness 0.3)))
+  )
+  (gr_text "VRLAB-KC" (at 183 52.5) (layer "F.SilkS")
+    (effects (font (size 1.5 1.5) (thickness 0.3)))
+  )
   (segment (start 140.88 59.085787) (end 140.88 71) (width 0.8) (layer "F.Cu") (net 1))
   (segment (start 134.38 54) (end 135.794213 54) (width 0.8) (layer "F.Cu") (net 1))
